File: pcb/GDEK.kicad_pcb (KiCad board)
At the start: 2 copper layers, 136.7 x 118 mm, 162 parts, among them J1 TYPE-C-31-M-13C, J2 AudioJack4, SW1 SW_Push_45deg, SW10 SW_Push_45deg, SW11 SW_Push_45deg, SW12 SW_Push_45deg, SW13 SW_Push_45deg, SW14 SW_Push_45deg, SW15 SW_Push_45deg, SW16 SW_Push_45deg, SW17 SW_Push_45deg, SW18 SW_Push_45deg, SW19 SW_Push_45deg, SW2 SW_Push_45deg, SW20 SW_Push_45deg, SW21 SW_Push_45deg, SW22 SW_Push_45deg, SW23 SW_Push_45deg, SW24 SW_Push_45deg, SW25 SW_Push_45deg, SW26 SW_Push_45deg, SW27 SW_Push_45deg, SW28 SW_Push_45deg, SW29 SW_Push_45deg, SW3 SW_Push_45deg, SW30 SW_Push_45deg, SW31 RotaryEncoder_Switch, SW4 SW_Push_45deg, SW5 SW_Push_45deg, SW6 SW_Push_45deg, SW7 SW_Push_45deg, SW8 SW_Push_45deg, SW9 SW_Push_45deg, U1 RP2040, U2 W25Q128JVS, U3 74AHCT1G125, U4 USBLC6-2P6, U5 XC6210B332MR, Y1 ABM8-272-T3

Commit message: 🚧 Start moving components and traces near USB connector
Parts:
- moved R9 11.1 mm to (141.4, 33.4)
- moved C17 11.1 mm to (137.4, 34.5)
- moved R8 11.1 mm to (137.4, 32.2)
- moved U3 11.1 mm to (135.2, 33.5)
- moved U4 11.1 mm to (139.4, 33.4)
- moved U5 11.1 mm to (144.4, 33.5)
Routing:
- net VBUS: track 22.8 -> 10.6 mm
- net GND: track 37.1 -> 28.1 mm, vias 12 -> 8
- net Net-(F1-Pad1): track 13.6 -> 8.25 mm
